Commit message: add comment for spring_stiffness

File: obinata_research/obinata_pr2_73b2_cleanup/models/room73b2-door-left/model.urdf.xacro (robot description, xacro)
@@ -51,4 +51,5 @@
       <mu2>0.9</mu2>
     </gazebo>
+    <!-- modify these params to make auto closing door? -->
     <joint name="${name}_root_parent_joint" type="fixed">
       <parent link="${parent}"/>
@@ -62,5 +63,6 @@
       <axis xyz="0 0 1"/>
       <limit lower="0" upper="1.5708" effort="100" velocity="0.5"/>
-      <dynamics damping="0.2" friction="0"/>
+      <!-- modify this param? -->
+      <dynamics damping="0.2" friction="0" spring_stiffness="0.5"/>
     </joint>
     <transmission type="pr2_mechanism_model/SimpleTransmission" name="${name}_DOOR_trans">

File: obinata_research/obinata_pr2_73b2_cleanup/models/room73b2-door-right/model.urdf.xacro (robot description, xacro)
@@ -28,4 +28,5 @@
       <mu2>0.9</mu2>
     </gazebo>
+    <!-- here? -->
     <link name="${name}_ROOM73B2-DOOR-RIGHT-BODYSET3_link">
       <visual>
@@ -102,4 +103,5 @@
       <insert_block name="origin"/>
     </joint>
+    <!-- here? -->
     <joint name="${name}_DOOR" type="revolute">
       <parent link="${name}_ROOM73B2-DOOR-RIGHT-BODYSET2_link"/>
@@ -108,5 +110,6 @@
       <axis xyz="0 0 -1"/>
       <limit lower="0" upper="1.5708" effort="100" velocity="0.5"/>
-      <dynamics damping="0.2" friction="0"/>
+      <!-- change spring_stiffness -->
+      <dynamics damping="0.2" friction="0" spring_stiffness="10000" />
     </joint>
     <transmission type="pr2_mechanism_model/SimpleTransmission" name="${name}_DOOR_trans">

File: obinata_research/obinata_pr2_73b2_cleanup/worlds/door_with_wall.urdf.xacro (robot description, xacro)
@@ -15,9 +15,9 @@
     </gazebo>
     <!-- door model -->
-    <xacro:include filename="$(find eusurdf)/models/room73b2-door-left/model.urdf.xacro"/>
+    <xacro:include filename="$(find obinata_pr2_73b2_cleanup)/models/room73b2-door-left/model.urdf.xacro"/>
     <room73b2-door-left name="room73b2-door-left_0" parent="room73b2_root_link">
         <origin xyz="0.0 0.405 0.0" rpy="0.0 0.0 0.0"/>
     </room73b2-door-left>
-    <xacro:include filename="$(find eusurdf)/models/room73b2-door-right/model.urdf.xacro"/>
+    <xacro:include filename="$(find obinata_pr2_73b2_cleanup)/models/room73b2-door-right/model.urdf.xacro"/>
     <room73b2-door-right name="room73b2-door-right_0" parent="room73b2_root_link">
         <origin xyz="0.0 -0.405 0.0" rpy="0.0 0.0 0.0"/>
