Commit message: fix style

File: obinata_research/obinata_pr2_73b2_cleanup/models/room73b2-door-right/model.urdf.xacro (robot description, xacro)
@@ -111,5 +111,5 @@
       <limit lower="0" upper="1.5708" effort="100" velocity="0.5"/>
       <!-- change spring_stiffness -->
-      <dynamics damping="0.2" friction="0" spring_stiffness="10000" />
+      <dynamics damping="0.2" friction="0" spring_stiffness="100.0" spring_reference="0.0" />
     </joint>
     <transmission type="pr2_mechanism_model/SimpleTransmission" name="${name}_DOOR_trans">

Commit message: modify tag style

File: obinata_research/obinata_pr2_73b2_cleanup/models/room73b2-door-right/model.urdf.xacro (robot description, xacro)
@@ -108,8 +108,19 @@
       <child link="${name}_ROOM73B2-DOOR-RIGHT-BODYSET3_link"/>
       <origin xyz="-0.015 -0.39 0" rpy="0 -0 0 "/>
-      <axis xyz="0 0 -1"/>
-      <limit lower="0" upper="1.5708" effort="100" velocity="0.5"/>
+      <axis>
+        <limit>
+          <lower>0</lower>
+          <upper>1.5708</upper>
+          <effort>100</effort>
+          <velocity>0.5</velocity>
+        </limit>
+        <xyz>0 0 1</xyz>
       <!-- change spring_stiffness -->
-      <dynamics damping="0.2" friction="0" spring_stiffness="100.0" spring_reference="0.0" />
+        <dynamics>
+          <damping>0.2</damping>
+          <friction>0</friction>
+          <spring_stiffness>100</spring_stiffness>
+        </dynamics>
+      </axis>
     </joint>
     <transmission type="pr2_mechanism_model/SimpleTransmission" name="${name}_DOOR_trans">

Commit message: succeeded in modifing springStiffness

File: obinata_research/obinata_pr2_73b2_cleanup/models/room73b2-door-right/model.urdf.xacro (robot description, xacro)
@@ -110,6 +110,5 @@
       <axis xyz="0 0 -1"/>
       <limit lower="0" upper="1.5708" effort="100" velocity="0.5"/>
-      <!-- change spring_stiffness -->
-      <dynamics damping="0.2" friction="0" spring_stiffness="100.0" spring_reference="0.0" />
+      <dynamics damping="0.2" friction="0"/>
     </joint>
     <transmission type="pr2_mechanism_model/SimpleTransmission" name="${name}_DOOR_trans">
@@ -118,5 +117,7 @@
       <mechanicalReduction>1</mechanicalReduction>
     </transmission>
+    <!-- modify springStiffness and make the door auto-closed -->
     <gazebo reference="${name}_DOOR">
+      <springStiffness>0.5</springStiffness>
       <cfmDamping>0.4</cfmDamping>
     </gazebo>
